Commit message: Working Hardware abstraction

File: hexapod_description/urdf/hexapod.urdf.xacro (robot description, xacro)
@@ -166,4 +166,19 @@
 		<material name="green"/>
 	</link>
+	<link name="front_marker">
+		<collision>
+			<geometry>
+				<box size="0.05 .05 .05" />
+			</geometry>
+			<origin xyz="-0.025 0 0" />
+		</collision>
+		<visual>
+			<geometry>
+				<box size="0.025 .025 .025" />
+			</geometry>
+			<origin xyz="-0.0125 0 0" />
+		</visual>
+		<material name="black"/>
+	</link>
 	<gazebo reference="base_link">
 	  	<material>Gazebo/Green</material>
@@ -171,4 +186,14 @@
 		<mu2>100</mu2>
 	</gazebo>
+	<gazebo reference="front_marker">
+	  	<material>Gazebo/Black</material>
+		<mu1>100</mu1>
+		<mu2>100</mu2>
+	</gazebo>
+	<joint name="front_marker_joint" type="fixed">
+		<parent link="base_link"/>
+		<child link="front_marker"/>
+		<origin xyz="0.2 0 0"/>
+	</joint>
 	<link name="inertial_sub">
 		<collision>

Commit message: added pycontroller

File: hexapod_description/urdf/hexapod.urdf.xacro (robot description, xacro)
@@ -7,5 +7,5 @@
 	  </plugin>
 	</gazebo>
-	<xacro:property name="upper_leg_length" value=".055" />
+	<xacro:property name="upper_leg_length" value=".053" />
 	<xacro:property name="lower_leg_length" value=".088" />
 	<material name="blue">
@@ -29,7 +29,7 @@
 												izz="${mass/12*(width*width+height*height)}" />
 											 -->
-			<inertia	ixx="1E-5" 	ixy="0.0" 	ixz="0.0"
-									iyy="1E-5" 	iyz="0.0"
-												izz="1E-5" />
+			<inertia	ixx="1E-3" 	ixy="0.0" 	ixz="0.0"
+									iyy="1E-3" 	iyz="0.0"
+												izz="1E-3" />
 		</inertial>
 	</xacro:macro>
@@ -38,5 +38,5 @@
 			<collision>
 				<geometry>
-					<box size="0.004 0.01 0.01" />
+					<box size="0.004 0.012 0.004" />
 				</geometry>
 				<origin xyz="0 ${reflect*0.005} 0" />
@@ -44,10 +44,10 @@
 			<visual>
 				<geometry>
-					<box size="0.004 0.01 0.01" />
+					<box size="0.004 0.012 0.004" />
 				</geometry>
 				<origin xyz="0 ${reflect*0.005} 0" />
 				<material name="black"/>
 			</visual>
-			<xacro:cube_inertial origin_xyz="0 ${reflect*0.005} 0" mass="0.01" width="0.004" height="0.01" depth="0.01"/>
+			<xacro:cube_inertial origin_xyz="0 ${reflect*0.005} 0" mass="0.025" width="0.004" height="0.01" depth="0.01"/>
 		</link>
 		<gazebo reference="${name}_coxa">
@@ -57,5 +57,5 @@
 			<collision>
 				<geometry>
-					<box size="0.004 ${upper_leg_length} 0.01" />
+					<box size="0.004 ${upper_leg_length} 0.004" />
 				</geometry>
 				<origin xyz="0 ${reflect*upper_leg_length/2} 0" />
@@ -63,10 +63,10 @@
 			<visual>
 				<geometry>
-					<box size="0.004 ${upper_leg_length} 0.01" />
+					<box size="0.004 ${upper_leg_length} 0.004" />
 				</geometry>
 				<material name="blue"/>
 				<origin xyz="0 ${reflect*upper_leg_length/2} 0" />
 			</visual>
-			<xacro:cube_inertial origin_xyz="0 ${reflect*upper_leg_length/2} 0" mass="0.01" width="0.004" height="${upper_leg_length}" depth="0.01"/>
+			<xacro:cube_inertial origin_xyz="0 ${reflect*upper_leg_length/2} 0" mass="0.025" width="0.004" height="${upper_leg_length}" depth="0.01"/>
 		</link>
 		<gazebo reference="${name}_femur">
@@ -76,5 +76,5 @@
 			<collision>
 				<geometry>
-					<box size="0.004 ${lower_leg_length} 0.01" />
+					<box size="0.004 ${lower_leg_length} 0.004" />
 				</geometry>
 				<origin xyz="0 ${reflect*lower_leg_length/2} 0" />
@@ -82,10 +82,10 @@
 			<visual>
 				<geometry>
-					<box size="0.004 ${lower_leg_length} 0.01" />
+					<box size="0.004 ${lower_leg_length} 0.004" />
 				</geometry>
 				<material name="red"/>
 				<origin xyz="0 ${reflect*lower_leg_length/2} 0" />
 			</visual>
-			<xacro:cube_inertial origin_xyz="0 ${reflect*lower_leg_length/2} 0" mass="0.01" width="0.004" height="${lower_leg_length}" depth="0.01"/>
+			<xacro:cube_inertial origin_xyz="0 ${reflect*lower_leg_length/2} 0" mass="0.015" width="0.004" height="${lower_leg_length}" depth="0.01"/>
 		</link>
 		<gazebo reference="${name}_tibia">
@@ -98,9 +98,10 @@
 		</gazebo>
 		<joint name="base_to_${name}_coxa" type="revolute">
-			<axis xyz="0 0 ${reflect*1}" />
-			<limit effort="2000" lower="-0.78" upper="0.78" velocity="0.5" />
+			<axis xyz="0 0 ${reflect*1}"/>
+			<dynamics damping=".05" friction=".05"/>
+			<limit effort="0.22" lower="-0.78" upper="0.78" velocity="10" />
 			<parent link="base_link" />
 			<child link="${name}_coxa" />
-			<origin xyz="${yoffset} ${reflect*0.04} 0.009" />
+			<origin xyz="${yoffset} ${reflect*0.0315} 0.005" />
 		</joint>
 		<transmission name="base_to_${name}_coxa_transmission">
@@ -115,8 +116,9 @@
 		<joint name="${name}_coxa_to_femur" type="revolute">
 			<axis xyz="${reflect*1} 0 0" />
-			<limit effort="2000" lower="-0.25" upper="1.5" velocity="0.5" />
+			<dynamics damping=".05" friction=".05"/>
+			<limit effort="0.22" lower="-0.25" upper="1.5" velocity="10" />
 			<parent link="${name}_coxa" />
 			<child link="${name}_femur" />
-			<origin xyz="0.004 ${reflect*0.01} 0" />
+			<origin xyz="0.004 ${reflect*0.012} 0" />
 		</joint>
 		<transmission name="coxa_to_${name}_femur_transmission">
@@ -131,8 +133,9 @@
 		<joint name="${name}_femur_to_tibia" type="revolute">
 			<axis xyz="${reflect*1} 0 0" />
-			<limit effort="2000" lower="-2.6" upper="0.5" velocity="0.5" />
+			<dynamics damping=".05" friction=".05"/>
+			<limit effort="0.22" lower="-2.6" upper="0.5" velocity="10" />
 			<parent link="${name}_femur" />
 			<child link="${name}_tibia" />
-			<origin xyz="0.004 ${reflect*upper_leg_length} 0" />
+			<origin xyz="0.000 ${reflect*upper_leg_length} 0" />
 		</joint>
 		<transmission name="femur_to_${name}_tibia_transmission">
@@ -146,20 +149,13 @@
 		</transmission>
 	</xacro:macro>
-	<!--
-	<link name="world"/>
-	<joint name="fixed" type="fixed">
-	  <parent link="world"/>
-	  <child link="base_link"/>
-	</joint>
- -->
 	<link name="base_link">
 		<collision>
 			<geometry>
-				<box size="0.2 .08 .05" />
+				<box size="0.115 .063 .05" />
 			</geometry>
 		</collision>
 		<visual>
 			<geometry>
-				<box size="0.2 .08 .05" />
+				<box size="0.115 .063 .05" />
 			</geometry>
 		</visual>
@@ -169,7 +165,7 @@
 		<collision>
 			<geometry>
-				<box size="0.05 .05 .05" />
-			</geometry>
-			<origin xyz="-0.025 0 0" />
+				<box size="0.02 .02 .02" />
+			</geometry>
+			<origin xyz="-0.01 0 0" />
 		</collision>
 		<visual>
@@ -194,18 +190,18 @@
 		<parent link="base_link"/>
 		<child link="front_marker"/>
-		<origin xyz="0.2 0 0"/>
+		<origin xyz="0.05 0 0.025"/>
 	</joint>
 	<link name="inertial_sub">
 		<collision>
 			<geometry>
-				<box size="0.2 .08 .05" />
+				<box size="0.115 .063 .05" />
 			</geometry>
 		</collision>
 		<visual>
 			<geometry>
-				<box size="0.2 .08 .05" />
+				<box size="0.115 .063 .05" />
 			</geometry>
 		</visual>
-		<xacro:cube_inertial origin_xyz="0 0 0" mass="0.05" width="0.2" height="0.08" depth="0.05"/>
+		<xacro:cube_inertial origin_xyz="0 0 0" mass="0.35" width="0.2" height="0.08" depth="0.05"/>
 	</link>
 	<gazebo reference="inertial_sub">
@@ -216,9 +212,9 @@
 		<child link="inertial_sub"/>
 	</joint>
-	<xacro:leg name="fl" yoffset="0.1" reflect="1" />
+	<xacro:leg name="fl" yoffset="0.0575" reflect="1" />
 	<xacro:leg name="ml" yoffset="0" reflect="1" />
-	<xacro:leg name="rl" yoffset="-0.1" reflect="1" />
-	<xacro:leg name="fr" yoffset="0.1" reflect="-1" />
+	<xacro:leg name="rl" yoffset="-0.0575" reflect="1" />
+	<xacro:leg name="fr" yoffset="0.0575" reflect="-1" />
 	<xacro:leg name="mr" yoffset="0" reflect="-1" />
-	<xacro:leg name="rr" yoffset="-0.1" reflect="-1" />
+	<xacro:leg name="rr" yoffset="-0.0575" reflect="-1" />
 </robot>

Commit message: First implementation of fielding's restrictedness walking

File: hexapod_description/urdf/hexapod.urdf.xacro (robot description, xacro)
@@ -100,5 +100,5 @@
 			<axis xyz="0 0 ${reflect*1}"/>
 			<dynamics damping=".05" friction=".05"/>
-			<limit effort="0.22" lower="-0.78" upper="0.78" velocity="10" />
+			<limit effort="0.35" lower="-0.78" upper="0.78" velocity="10" />
 			<parent link="base_link" />
 			<child link="${name}_coxa" />
@@ -117,5 +117,5 @@
 			<axis xyz="${reflect*1} 0 0" />
 			<dynamics damping=".05" friction=".05"/>
-			<limit effort="0.22" lower="-0.25" upper="1.5" velocity="10" />
+			<limit effort="0.35" lower="-0.25" upper="2.5" velocity="10" />
 			<parent link="${name}_coxa" />
 			<child link="${name}_femur" />
@@ -134,5 +134,5 @@
 			<axis xyz="${reflect*1} 0 0" />
 			<dynamics damping=".05" friction=".05"/>
-			<limit effort="0.22" lower="-2.6" upper="0.5" velocity="10" />
+			<limit effort="0.35" lower="-2.6" upper="0.5" velocity="10" />
 			<parent link="${name}_femur" />
 			<child link="${name}_tibia" />
